File: 555LEDs.kicad_pcb (KiCad board)
At the start: 2 copper layers, 89.4 x 72 mm, 18 parts, among them J1 Conn_01x02_Socket, U1 NE555P, U2 4017

Commit message: Add files via upload
Parts:
- RV1: footprint Potentiometer_THT:Potentiometer_Vishay_T93YA_Vertical -> Potentiometer_THT:Potentiometer_Alps_RK09K_Single_Vertical
- moved D5 22.3 mm to (187.0, 64.1)
- moved D3 21.7 mm to (126.1, 96.0)
- moved D7 21.7 mm to (171.3, 118.8)
- moved D8 21.7 mm to (209.7, 96.8)
- moved R1 21.7 mm to (136.6, 99.2)
- moved U2 21.7 mm to (170.6, 88.1)
- moved C2 21.7 mm to (204.8, 105.8)
- moved D2 21.7 mm to (143.0, 60.7)
- moved D4 21.7 mm to (208.3, 82.2)
- moved D6 21.7 mm to (161.0, 55.1)
- moved D9 21.7 mm to (203.0, 66.9)
- moved J1 21.7 mm to (132.0, 114.3)
- moved U1 21.7 mm to (170.2, 100.6)
- moved D10 21.7 mm to (174.0, 64.5)
- moved C1 21.7 mm to (155.6, 114.6)
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Routing:
- net +5V: track 122.6 -> 102.2 mm
- net (no net): track 16.6 -> 0.62 mm, vias 2 -> 0
- net Net-(U1-THRES): track 56.7 -> 42.6 mm, vias 0 -> 2
- net Net-(U1-DISCH): track 91.7 -> 83.5 mm
- net Net-(D1-K): track 0.30 -> 2.91 mm, vias 0 -> 2
- net Net-(D8-A): track 58.4 -> 60.0 mm
- net Net-(D9-A): track 48.8 -> 49.8 mm
- net Net-(D5-A): track 39.1 -> 38.3 mm
- net Net-(D4-A): track 59.4 -> 60.1 mm, vias 0 -> 1
Other:
- board text added: "Philipp Buda 16.10.2026"
