File: 555LEDs.kicad_sch (KiCad schematic)
At the start: 18 parts, among them J1 Conn_01x02_Socket, U1 NE555P, U2 4017

Commit message: Add files via upload
Parts:
- RV1: footprint Potentiometer_THT:Potentiometer_Vishay_T93YA_Vertical -> Potentiometer_THT:Potentiometer_Alps_RK09K_Single_Vertical
Changed lines of the file:
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@@
 			)
 		)
-		(property "Footprint" "Potentiometer_THT:Potentiometer_Vishay_T93YA_Vertical"
+		(property "Footprint" "Potentiometer_THT:Potentiometer_Alps_RK09K_Single_Vertical"
 			(at 64.77 40.64 0)
 			(hide yes)
